Commit message: Add base_link collider (box) for recovery; verified walking unchanged
Recovery needs real torso–floor contact for fallen-pose physics. The full
base_link visual mesh would penetrate hip_yaw/hip_roll meshes by ~9cm at
rest (CAD components physically share housing), so we use a box primitive
sized to the upper torso (above the hip mount) — clears all hip meshes by
8cm and matches the actual contactable torso shell.

- assets/q1/urdf/q1.urdf: add <collision> box (0.32 x 0.22 x 0.12 @ z=0.05)
- deploy/sim2sim/sim2sim.py: drop now-dead URDF string patch + base_link
  disable workaround; URDF is the single source of truth
- configs/recovery.yaml: enable terminal layer + soften height/orientation
  exp coefficients (k_h: 30 -> 2, k_o: 2 -> 0.2) for gradient from fallen
- env/tasks/recovery_task.py: read height_k / orientation_k from config

Verified:
- BIRL bdx_slim_v3 sim2sim walking unchanged (z=0.37, pitch +/-2 deg)
- No self-collision contacts at rest pose

File: assets/q1/urdf/q1.urdf (robot description, URDF)
Before this commit: robot YSXSZ, 12 links, 11 joints
Links:
- link base_link: geometry collision box size=0.32 0.22 0.12; visual mesh filename=../meshes/base_link.STL
